File: PID Toaster/PID Toaster.kicad_pcb (KiCad board)
At the start: 2 copper layers, 105 parts, among them J1 Conn_01x02_Socket, J2 Conn_01x03_Socket, J3 Conn_01x02_Socket, J4 AVR-JTAG-10, J5 Conn_01x03_Socket, J6 Conn_01x08_Socket, J7 Conn_01x02_Socket, J8 Conn_01x02_Socket, J9 Micro_SD_Card, P1 USB_C_Plug_USB2.0, Q1 NPN, Q2 PNP, Q3 NPN, Q4 PNP, SW1 SW_Push, SW10 SW_Push, SW11 SW_Push, SW12 SW_Push, SW13 SW_Push, SW14 SW_Push, SW15 SW_Push, SW16 SW_Push, SW17 SW_Push, SW18 SW_Push, SW2 SW_Push, SW3 SW_Push, SW4 SW_Push, SW5 SW_Push, SW6 SW_Push, SW7 SW_Push, SW8 SW_Push, SW9 SW_Push, U1 W25Q128JVS, U2 RP2350A-QFN60, U3 AMS1117, U4 NCP1117-3.3_SOT223, U5 MAX31855KASA, U6 MAX31855KASA, Y1 12MHz

Commit message: update
Parts:
- moved C15 46.1 mm to (18.3, 84.0)
- moved Q3 46.1 mm to (23.2, 82.5)
- moved Q4 46.1 mm to (23.2, 87.2)
- moved R7 46.1 mm to (23.1, 78.9)
- moved R11 46.1 mm to (23.1, 90.7)
- moved C19 18.7 mm to (106.2, 54.4)
- moved U3 18.7 mm to (106.2, 62.1)
- moved D3 17.2 mm to (106.0, 68.5), turned to 0 degrees
- moved J3 12.3 mm to (54.9, 51.6), turned to 90 degrees
- moved PS1 9.87 mm to (67.5, 56.5)
- moved U5 8.78 mm to (62.9, 79.6)
- moved U6 8.78 mm to (62.9, 73.0)
- moved J1 8.74 mm to (112.5, 47.8)
- moved J2 3.50 mm to (61.4, 99.3)
- moved J5 3.50 mm to (51.2, 99.3)
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Other:
- board outline added: 76.6 x 143.7 mm
